Commit message: edit: file structure; motoman_moveit & motoman_support directories created to house large volume of repos for organization, some filepaths corrected; WIP

File: motoman_description/arms/gp7/urdf/gp7.urdf.xacro (robot description, xacro)
@@ -1,6 +1,6 @@
 <?xml version="1.0"?>
 <robot xmlns:xacro="http://ros.org/wiki/xacro">
-  <xacro:include filename="$(find motoman_gp7_support)/urdf/gp7.transmission.xacro" />
-  <xacro:include filename="$(find motoman_gp7_support)/urdf/gp7.gazebo.xacro" />
+  <xacro:include filename="$(find motoman_description)/arms/gp7/urdf/gp7.transmission.xacro" />
+  <xacro:include filename="$(find motoman_description)/arms/gp7/urdf/gp7.gazebo.xacro" />
   <xacro:macro name="gp7_robot" params="prefix">
     <!-- Properties -->
@@ -12,5 +12,5 @@
         <visual>
             <geometry>
-                <mesh filename="package://motoman_gp7_support/meshes/visual/gp7_base_link.stl"/>
+                <mesh filename="package://motoman_description/arms/gp7/meshes/visual/gp7_base_link.stl"/>
             </geometry>
             <material name="yaskawa_blue"/>
@@ -18,5 +18,5 @@
         <collision>
             <geometry>
-                <mesh filename="package://motoman_gp7_support/meshes/collision/gp7_base_link.stl"/>
+                <mesh filename="package://motoman_description/arms/gp7/meshes/collision/gp7_base_link.stl"/>
             </geometry>
         </collision>
@@ -25,5 +25,5 @@
         <visual>
             <geometry>
-                <mesh filename="package://motoman_gp7_support/meshes/visual/gp7_link_1_s.stl"/>
+                <mesh filename="package://motoman_description/arms/gp7/meshes/visual/gp7_link_1_s.stl"/>
             </geometry>
             <material name="yaskawa_blue"/>
@@ -31,5 +31,5 @@
         <collision>
             <geometry>
-                <mesh filename="package://motoman_gp7_support/meshes/collision/gp7_link_1_s.stl"/>
+                <mesh filename="package://motoman_description/arms/gp7/meshes/collision/gp7_link_1_s.stl"/>
             </geometry>
         </collision>
@@ -38,5 +38,5 @@
         <visual>
             <geometry>
-                <mesh filename="package://motoman_gp7_support/meshes/visual/gp7_link_2_l.stl"/>
+                <mesh filename="package://motoman_description/arms/gp7/meshes/visual/gp7_link_2_l.stl"/>
             </geometry>
             <material name="yaskawa_blue"/>
@@ -44,5 +44,5 @@
         <collision>
             <geometry>
-                <mesh filename="package://motoman_gp7_support/meshes/collision/gp7_link_2_l.stl"/>
+                <mesh filename="package://motoman_description/arms/gp7/meshes/collision/gp7_link_2_l.stl"/>
             </geometry>
         </collision>
@@ -51,5 +51,5 @@
         <visual>
             <geometry>
-                <mesh filename="package://motoman_gp7_support/meshes/visual/gp7_link_3_u.stl"/>
+                <mesh filename="package://motoman_description/arms/gp7/meshes/visual/gp7_link_3_u.stl"/>
             </geometry>
             <material name="yaskawa_blue"/>
@@ -57,5 +57,5 @@
         <collision>
             <geometry>
-                <mesh filename="package://motoman_gp7_support/meshes/collision/gp7_link_3_u.stl"/>
+                <mesh filename="package://motoman_description/arms/gp7/meshes/collision/gp7_link_3_u.stl"/>
             </geometry>
         </collision>
@@ -64,5 +64,5 @@
         <visual>
             <geometry>
-                <mesh filename="package://motoman_gp7_support/meshes/visual/gp7_link_4_r.stl"/>
+                <mesh filename="package://motoman_description/arms/gp7/meshes/visual/gp7_link_4_r.stl"/>
             </geometry>
             <material name="yaskawa_blue"/>
@@ -70,5 +70,5 @@
         <collision>
             <geometry>
-                <mesh filename="package://motoman_gp7_support/meshes/collision/gp7_link_4_r.stl"/>
+                <mesh filename="package://motoman_description/arms/gp7/meshes/collision/gp7_link_4_r.stl"/>
             </geometry>
         </collision>
@@ -77,5 +77,5 @@
         <visual>
             <geometry>
-                <mesh filename="package://motoman_gp7_support/meshes/visual/gp7_link_5_b.stl"/>
+                <mesh filename="package://motoman_description/arms/gp7/meshes/visual/gp7_link_5_b.stl"/>
             </geometry>
             <material name="yaskawa_blue"/>
@@ -83,5 +83,5 @@
         <collision>
             <geometry>
-                <mesh filename="package://motoman_gp7_support/meshes/collision/gp7_link_5_b.stl"/>
+                <mesh filename="package://motoman_description/arms/gp7/meshes/collision/gp7_link_5_b.stl"/>
             </geometry>
         </collision>
@@ -90,5 +90,5 @@
         <visual>
             <geometry>
-                <mesh filename="package://motoman_gp7_support/meshes/visual/gp7_link_6_t.stl"/>
+                <mesh filename="package://motoman_description/arms/gp7/meshes/visual/gp7_link_6_t.stl"/>
             </geometry>
             <material name="yaskawa_blue"/>
@@ -96,5 +96,5 @@
         <collision>
             <geometry>
-                <mesh filename="package://motoman_gp7_support/meshes/collision/gp7_link_6_t.stl"/>
+                <mesh filename="package://motoman_description/arms/gp7/meshes/collision/gp7_link_6_t.stl"/>
             </geometry>
         </collision>

File: motoman_description/arms/gp7/urdf/gp7_robot.urdf.xacro (robot description, xacro)
@@ -3,7 +3,7 @@
        name="gp7" >
   <!-- common stuff -->
-  <xacro:include filename="$(find motoman_gp7_support)/urdf/common.gp7.xacro" />
+  <xacro:include filename="$(find motoman_description)/arms/gp7/urdf/common.gp7.xacro" />
   <!-- ur5e -->
-  <xacro:include filename="$(find motoman_gp7_support)/urdf/gp7.urdf.xacro" />
+  <xacro:include filename="$(find motoman_description)/arms/gp7/urdf/gp7.urdf.xacro" />
   <!-- arm -->
   <xacro:gp7_robot prefix="" />
