Commit message: edit: file structure to be consistent with other robot repositories, add: moveit confiurations for gp7 also with r2f85/140, add: arm_and_gripper group for controlling whole system

File: motoman_description/grippers/robotiq_2f_140/urdf/robotiq_2f_140_macro.xacro (robot description, xacro)
@@ -2,5 +2,5 @@
 <robot name="robotiq_arg2f_140_model" xmlns:xacro="http://ros.org/wiki/xacro">
   <xacro:macro name="load_gripper" params="parent prefix">
-    <xacro:include filename="$(find ur_e_description)/grippers/robotiq_2f_140/urdf/robotiq_arg2f_140_model_macro.xacro" />
+    <xacro:include filename="$(find motoman_description)/grippers/robotiq_2f_140/urdf/robotiq_arg2f_140_model_macro.xacro" />
     <xacro:robotiq_arg2f_140 parent="${parent}" prefix="${prefix}"/>
   </xacro:macro>

File: motoman_description/grippers/robotiq_2f_140/urdf/robotiq_2f_140_transmission_macro.xacro (robot description, xacro)
@@ -55,6 +55,6 @@
             <plugin name="gazebo_grasp_fix" filename="libgazebo_grasp_fix.so">
                 <arm>
-                    <arm_name>ur5e</arm_name>
-                    <palm_link>${prefix}wrist_3_link</palm_link>
+                    <arm_name>gp7</arm_name>
+                    <palm_link>${prefix}link_6_t</palm_link>
                     <!-- Gazebo merges links connected by fixed joints, so you need to check the links in gazebo and choose one that is recognized after internal connections are made. We would want to choose the actual paml of the gripper but it is currently not an option -->
                     <gripper_link> ${prefix}left_inner_finger </gripper_link>

File: motoman_description/grippers/robotiq_2f_140/urdf/robotiq_arg2f.xacro (robot description, xacro)
@@ -7,5 +7,5 @@
         <parent link="${parent}"/>
         <child link="${prefix}robotiq_arg2f_base_link"/>
-        <origin rpy="0.0 ${pi/2} 0.0" xyz="0.0 0.0 0.0"/>
+        <origin rpy="0.0 0.0 0.0" xyz="0.0 0.0 0.0"/>
     </joint>
     <link name="${prefix}robotiq_arg2f_base_link">
@@ -20,5 +20,5 @@
           <!-- The DAE file doesn't show well in Gazebo so we're using the STL instead -->
           <!-- <mesh filename="package://ur_e_description/grippers/robotiq_2f_140/meshes/visual/robotiq_arg2f_140_base_link.dae" scale="0.001 0.001 0.001"/> -->
-          <mesh filename="package://ur_e_description/grippers/robotiq_2f_140/meshes/collision/robotiq_arg2f_base_link.stl" />
+          <mesh filename="package://motoman_description/grippers/robotiq_2f_140/meshes/collision/robotiq_arg2f_base_link.stl" />
         </geometry>
         <material name="">
@@ -29,5 +29,5 @@
         <origin xyz="0 0 0" rpy="0 0 0" />
         <geometry>
-          <mesh filename="package://ur_e_description/grippers/robotiq_2f_140/meshes/collision/robotiq_arg2f_base_link.stl" />
+          <mesh filename="package://motoman_description/grippers/robotiq_2f_140/meshes/collision/robotiq_arg2f_base_link.stl" />
         </geometry>
       </collision>

File: motoman_description/grippers/robotiq_2f_140/urdf/robotiq_arg2f_140_model_macro.xacro (robot description, xacro)
@@ -17,5 +17,5 @@
         <origin xyz="0 0 0" rpy="0 0 0" />
         <geometry>
-          <mesh filename="package://ur_e_description/grippers/robotiq_2f_140/meshes/visual/robotiq_arg2f_${stroke}_outer_knuckle.stl" />
+          <mesh filename="package://motoman_description/grippers/robotiq_2f_140/meshes/visual/robotiq_arg2f_${stroke}_outer_knuckle.stl" />
         </geometry>
         <material name="">
@@ -26,5 +26,5 @@
         <origin xyz="0 0 0" rpy="0 0 0" />
         <geometry>
-          <mesh filename="package://ur_e_description/grippers/robotiq_2f_140/meshes/collision/robotiq_arg2f_${stroke}_outer_knuckle.stl" />
+          <mesh filename="package://motoman_description/grippers/robotiq_2f_140/meshes/collision/robotiq_arg2f_${stroke}_outer_knuckle.stl" />
         </geometry>
       </collision>
@@ -55,5 +55,5 @@
         <origin xyz="0 0 0" rpy="0 0 0" />
         <geometry>
-          <mesh filename="package://ur_e_description/grippers/robotiq_2f_140/meshes/visual/robotiq_arg2f_${stroke}_outer_finger.stl" />
+          <mesh filename="package://motoman_description/grippers/robotiq_2f_140/meshes/visual/robotiq_arg2f_${stroke}_outer_finger.stl" />
         </geometry>
         <material name="">
@@ -64,5 +64,5 @@
         <origin xyz="0 0 0" rpy="0 0 0" />
         <geometry>
-          <mesh filename="package://ur_e_description/grippers/robotiq_2f_140/meshes/collision/robotiq_arg2f_${stroke}_outer_finger.stl" />
+          <mesh filename="package://motoman_description/grippers/robotiq_2f_140/meshes/collision/robotiq_arg2f_${stroke}_outer_finger.stl" />
         </geometry>
       </collision>
@@ -88,5 +88,5 @@
         <origin xyz="0 0 0" rpy="0 0 0" />
         <geometry>
-          <mesh filename="package://ur_e_description/grippers/robotiq_2f_140/meshes/visual/robotiq_arg2f_${stroke}_inner_knuckle.stl" />
+          <mesh filename="package://motoman_description/grippers/robotiq_2f_140/meshes/visual/robotiq_arg2f_${stroke}_inner_knuckle.stl" />
         </geometry>
         <material name="">
@@ -97,5 +97,5 @@
         <origin xyz="0 0 0" rpy="0 0 0" />
         <geometry>
-          <mesh filename="package://ur_e_description/grippers/robotiq_2f_140/meshes/collision/robotiq_arg2f_${stroke}_inner_knuckle.stl" />
+          <mesh filename="package://motoman_description/grippers/robotiq_2f_140/meshes/collision/robotiq_arg2f_${stroke}_inner_knuckle.stl" />
         </geometry>
       </collision>
@@ -121,5 +121,5 @@
         <origin xyz="0 0 0" rpy="0 0 0" />
         <geometry>
-          <mesh filename="package://ur_e_description/grippers/robotiq_2f_140/meshes/visual/robotiq_arg2f_${stroke}_inner_finger.stl" />
+          <mesh filename="package://motoman_description/grippers/robotiq_2f_140/meshes/visual/robotiq_arg2f_${stroke}_inner_finger.stl" />
         </geometry>
         <material name="">
@@ -130,5 +130,5 @@
         <origin xyz="0 0 0" rpy="0 0 0" />
         <geometry>
-          <mesh filename="package://ur_e_description/grippers/robotiq_2f_140/meshes/collision/robotiq_arg2f_${stroke}_inner_finger.stl" />
+          <mesh filename="package://motoman_description/grippers/robotiq_2f_140/meshes/collision/robotiq_arg2f_${stroke}_inner_finger.stl" />
         </geometry>
       </collision>
@@ -197,5 +197,5 @@
     </joint>
   </xacro:macro>
-  <xacro:include filename="$(find ur_e_description)/grippers/robotiq_2f_140/urdf/robotiq_arg2f.xacro" />
+  <xacro:include filename="$(find motoman_description)/grippers/robotiq_2f_140/urdf/robotiq_arg2f.xacro" />
   <xacro:macro name="finger_joint" params="prefix">
     <joint name="${prefix}finger_joint" type="revolute">

File: motoman_description/grippers/robotiq_2f_85/urdf/robotiq_2f_85_macro.xacro (robot description, xacro)
@@ -2,5 +2,5 @@
 <robot name="robotiq_arg2f_85_model" xmlns:xacro="http://ros.org/wiki/xacro">
   <xacro:macro name="load_gripper" params="parent prefix">
-    <xacro:include filename="$(find ur_e_description)/grippers/robotiq_2f_85/urdf/robotiq_arg2f_85_model_macro.xacro" />
+    <xacro:include filename="$(find motoman_description)/grippers/robotiq_2f_85/urdf/robotiq_arg2f_85_model_macro.xacro" />
     <xacro:robotiq_arg2f_85 parent="${parent}" prefix="${prefix}"/>
   </xacro:macro>

File: motoman_description/grippers/robotiq_2f_85/urdf/robotiq_2f_85_transmission_macro.xacro (robot description, xacro)
@@ -55,6 +55,6 @@
             <plugin name="gazebo_grasp_fix" filename="libgazebo_grasp_fix.so">
                 <arm>
-                    <arm_name>ur5e</arm_name>
-                    <palm_link>${prefix}wrist_3_link</palm_link>
+                    <arm_name>gp7</arm_name>
+                    <palm_link>${prefix}link_6_t</palm_link>
                     <!-- Gazebo merges links connected by fixed joints, so you need to check the links in gazebo and choose one that is recognized after internal connections are made. We would want to choose the actual paml of the gripper but it is currently not an option -->
                     <gripper_link> ${prefix}left_inner_finger </gripper_link>

File: motoman_description/grippers/robotiq_2f_85/urdf/robotiq_arg2f.xacro (robot description, xacro)
@@ -7,5 +7,5 @@
         <parent link="${parent}"/>
         <child link="${prefix}robotiq_arg2f_base_link"/>
-        <origin rpy="0.0 ${pi/2} 0.0" xyz="0.0 0.0 0.0"/>
+        <origin rpy="0.0 0.0 0.0" xyz="0.0 0.0 0.0"/>
     </joint>
     <link name="${prefix}robotiq_arg2f_base_link">
@@ -20,5 +20,5 @@
           <!-- The DAE file doesn't show well in Gazebo so we're using the STL instead -->
           <!-- <mesh filename="package://kortex_description/grippers/robotiq_2f_85/meshes/visual/robotiq_arg2f_85_base_link.dae" scale="0.001 0.001 0.001"/> -->
-          <mesh filename="package://ur_e_description/grippers/robotiq_2f_85/meshes/collision/robotiq_arg2f_base_link.stl" />
+          <mesh filename="package://motoman_description/grippers/robotiq_2f_85/meshes/collision/robotiq_arg2f_base_link.stl" />
         </geometry>
         <material name="">
@@ -29,5 +29,5 @@
         <origin xyz="0 0 0" rpy="0 0 0" />
         <geometry>
-          <mesh filename="package://ur_e_description/grippers/robotiq_2f_85/meshes/collision/robotiq_arg2f_base_link.stl" />
+          <mesh filename="package://motoman_description/grippers/robotiq_2f_85/meshes/collision/robotiq_arg2f_base_link.stl" />
         </geometry>
       </collision>

File: motoman_description/grippers/robotiq_2f_85/urdf/robotiq_arg2f_85_model_macro.xacro (robot description, xacro)
@@ -11,5 +11,5 @@
         <origin xyz="0 0 0" rpy="0 0 0" />
         <geometry>
-          <mesh filename="package://ur_e_description/grippers/robotiq_2f_85/meshes/visual/robotiq_arg2f_85_outer_knuckle.dae" scale="0.001 0.001 0.001"/>
+          <mesh filename="package://motoman_description/grippers/robotiq_2f_85/meshes/visual/robotiq_arg2f_85_outer_knuckle.dae" scale="0.001 0.001 0.001"/>
         </geometry>
         <material name="">
@@ -20,5 +20,5 @@
         <origin xyz="0 0 0" rpy="0 0 0" />
         <geometry>
-          <mesh filename="package://ur_e_description/grippers/robotiq_2f_85/meshes/collision/robotiq_arg2f_85_outer_knuckle.dae" scale="0.001 0.001 0.001"/>
+          <mesh filename="package://motoman_description/grippers/robotiq_2f_85/meshes/collision/robotiq_arg2f_85_outer_knuckle.dae" scale="0.001 0.001 0.001"/>
         </geometry>
       </collision>
@@ -35,5 +35,5 @@
         <origin xyz="0 0 0" rpy="0 0 0" />
         <geometry>
-          <mesh filename="package://ur_e_description/grippers/robotiq_2f_85/meshes/visual/robotiq_arg2f_85_outer_finger.dae" scale="0.001 0.001 0.001"/>
+          <mesh filename="package://motoman_description/grippers/robotiq_2f_85/meshes/visual/robotiq_arg2f_85_outer_finger.dae" scale="0.001 0.001 0.001"/>
         </geometry>
         <material name="">
@@ -44,5 +44,5 @@
         <origin xyz="0 0 0" rpy="0 0 0" />
         <geometry>
-          <mesh filename="package://ur_e_description/grippers/robotiq_2f_85/meshes/collision/robotiq_arg2f_85_outer_finger.dae" scale="0.001 0.001 0.001"/>
+          <mesh filename="package://motoman_description/grippers/robotiq_2f_85/meshes/collision/robotiq_arg2f_85_outer_finger.dae" scale="0.001 0.001 0.001"/>
         </geometry>
       </collision>
@@ -59,5 +59,5 @@
         <origin xyz="0 0 0" rpy="0 0 0" />
         <geometry>
-          <mesh filename="package://ur_e_description/grippers/robotiq_2f_85/meshes/visual/robotiq_arg2f_85_inner_knuckle.dae" scale="0.001 0.001 0.001"/>
+          <mesh filename="package://motoman_description/grippers/robotiq_2f_85/meshes/visual/robotiq_arg2f_85_inner_knuckle.dae" scale="0.001 0.001 0.001"/>
         </geometry>
         <material name="">
@@ -68,5 +68,5 @@
         <origin xyz="0 0 0" rpy="0 0 0" />
         <geometry>
-          <mesh filename="package://ur_e_description/grippers/robotiq_2f_85/meshes/collision/robotiq_arg2f_85_inner_knuckle.dae" scale="0.001 0.001 0.001"/>
+          <mesh filename="package://motoman_description/grippers/robotiq_2f_85/meshes/collision/robotiq_arg2f_85_inner_knuckle.dae" scale="0.001 0.001 0.001"/>
         </geometry>
       </collision>
@@ -83,5 +83,5 @@
         <origin xyz="0 0 0" rpy="0 0 0" />
         <geometry>
-          <mesh filename="package://ur_e_description/grippers/robotiq_2f_85/meshes/visual/robotiq_arg2f_85_inner_finger.dae" scale="0.001 0.001 0.001"/>
+          <mesh filename="package://motoman_description/grippers/robotiq_2f_85/meshes/visual/robotiq_arg2f_85_inner_finger.dae" scale="0.001 0.001 0.001"/>
         </geometry>
         <material name="">
@@ -92,5 +92,5 @@
         <origin xyz="0 0 0" rpy="0 0 0" />
         <geometry>
-          <mesh filename="package://ur_e_description/grippers/robotiq_2f_85/meshes/collision/robotiq_arg2f_85_inner_finger.dae" scale="0.001 0.001 0.001" />
+          <mesh filename="package://motoman_description/grippers/robotiq_2f_85/meshes/collision/robotiq_arg2f_85_inner_finger.dae" scale="0.001 0.001 0.001" />
         </geometry>
       </collision>
@@ -157,5 +157,5 @@
     </joint>
   </xacro:macro>
-  <xacro:include filename="$(find ur_e_description)/grippers/robotiq_2f_85/urdf/robotiq_arg2f.xacro" />
+  <xacro:include filename="$(find motoman_description)/grippers/robotiq_2f_85/urdf/robotiq_arg2f.xacro" />
   <xacro:macro name="finger_joint" params="prefix">
     <joint name="${prefix}finger_joint" type="revolute">
