Commit message: edit: robot_workstation description files to actually include workstation, fix: launch file not calling proper robot description files

File: motoman_description/urdf/gp7_robot_robotiq_2f_140_workstation.urdf.xacro (robot description, xacro)
@@ -6,11 +6,27 @@
   <!-- gp7 -->
   <xacro:include filename="$(find motoman_description)/urdf/gp7.urdf.xacro" />
+  <!-- ARMada workstation -->
+  <xacro:include filename="$(find uml_hri_nerve_armada_workstation)/workstation_description/workstation_model.urdf.xacro" />
+  <!-- robotiq_2f_140 -->
+  <xacro:include filename="$(find motoman_description)/grippers/robotiq_2f_140/urdf/robotiq_2f_140_macro.xacro" />
+  <xacro:include filename="$(find motoman_description)/grippers/robotiq_2f_140/urdf/robotiq_2f_140_transmission_macro.xacro" />
   <!-- arm -->
   <xacro:motoman_gp7 prefix="" />
+  <!-- gripper -->
+  <xacro:load_gripper parent="tool0"  prefix=""/>
+  <xacro:load_gazebo_gripper_transmissions prefix=""/>
+  <!-- workstation -->
+  <xacro:workstation prefix="table_" namespace=""/>
   <link name="world" />
-  <joint name="world_joint" type="fixed">
+  <joint name="connect_world_and_table" type="fixed">
+    <child link="table_base_link" />
     <parent link="world" />
+    <origin xyz="0.0 0.0 0.41" rpy="0.0 0.0 0.0" />
+  </joint>
+  <!-- needs to be like kinova where root link is an argument -->
+  <joint name="connect_table_and_arm" type="fixed">
+    <parent link="table_mounting_plate_link" />
     <child link = "base_link" />
-    <origin xyz="0.0 0.0 0.0" rpy="0.0 0.0 0.0" />
+    <origin xyz="0.0 0.0 0.03625" rpy="0.0 0.0 ${pi/2}" />
   </joint>
 </robot>

File: motoman_description/urdf/gp7_robot_robotiq_2f_85_workstation.urdf.xacro (robot description, xacro)
@@ -6,11 +6,27 @@
   <!-- gp7 -->
   <xacro:include filename="$(find motoman_description)/urdf/gp7.urdf.xacro" />
+  <!-- ARMada workstation -->
+  <xacro:include filename="$(find uml_hri_nerve_armada_workstation)/workstation_description/workstation_model.urdf.xacro" />
+  <!-- robotiq_2f_85 -->
+  <xacro:include filename="$(find motoman_description)/grippers/robotiq_2f_85/urdf/robotiq_2f_85_macro.xacro" />
+  <xacro:include filename="$(find motoman_description)/grippers/robotiq_2f_85/urdf/robotiq_2f_85_transmission_macro.xacro" />
   <!-- arm -->
   <xacro:motoman_gp7 prefix="" />
+  <!-- gripper -->
+  <xacro:load_gripper parent="tool0"  prefix=""/>
+  <xacro:load_gazebo_gripper_transmissions prefix=""/>
+  <!-- workstation -->
+  <xacro:workstation prefix="table_" namespace=""/>
   <link name="world" />
-  <joint name="world_joint" type="fixed">
+  <joint name="connect_world_and_table" type="fixed">
+    <child link="table_base_link" />
     <parent link="world" />
+    <origin xyz="0.0 0.0 0.41" rpy="0.0 0.0 0.0" />
+  </joint>
+  <!-- needs to be like kinova where root link is an argument -->
+  <joint name="connect_table_and_arm" type="fixed">
+    <parent link="table_mounting_plate_link" />
     <child link = "base_link" />
-    <origin xyz="0.0 0.0 0.0" rpy="0.0 0.0 0.0" />
+    <origin xyz="0.0 0.0 0.03625" rpy="0.0 0.0 ${pi/2}" />
   </joint>
 </robot>

File: motoman_description/urdf/gp7_robot_workstation.urdf.xacro (robot description, xacro)
@@ -6,11 +6,21 @@
   <!-- gp7 -->
   <xacro:include filename="$(find motoman_description)/urdf/gp7.urdf.xacro" />
+  <!-- ARMada workstation -->
+  <xacro:include filename="$(find uml_hri_nerve_armada_workstation)/workstation_description/workstation_model.urdf.xacro" />
   <!-- arm -->
   <xacro:motoman_gp7 prefix="" />
+  <!-- workstation -->
+  <xacro:workstation prefix="table_" namespace=""/>
   <link name="world" />
-  <joint name="world_joint" type="fixed">
+  <joint name="connect_world_and_table" type="fixed">
+    <child link="table_base_link" />
     <parent link="world" />
+    <origin xyz="0.0 0.0 0.41" rpy="0.0 0.0 0.0" />
+  </joint>
+  <!-- needs to be like kinova where root link is an argument -->
+  <joint name="connect_table_and_arm" type="fixed">
+    <parent link="table_mounting_plate_link" />
     <child link = "base_link" />
-    <origin xyz="0.0 0.0 0.0" rpy="0.0 0.0 0.0" />
+    <origin xyz="0.0 0.0 0.03625" rpy="0.0 0.0 ${pi/2}" />
   </joint>
 </robot>
